File: TPS5430_Buck_5V.kicad_sch (KiCad schematic)
At the start: 20 parts, among them J1 Barrel_Jack, J2 Conn_01x02_Pin, U1 TPS54308

Commit message: add barrel jack symbol,footprint and 3d model and rough placement
Parts:
- removed J1: Barrel_Jack, symbol Connector:Barrel_Jack
- added J1: 694103107102, Connector_SMD_Wurth:J_Wurth_WR-DC_694103107102, symbol Barrel-Jack:694103107102
- C1, C2, C3, C4, C5, C6: footprint (none) -> Capacitor_SMD:C_0805_2012Metric
- H1, H2, H3, H4: footprint (none) -> MountingHole:MountingHole_2.2mm_M2_ISO7380
- J2: footprint (none) -> Connector_PinHeader_1.00mm:PinHeader_1x02_P1.00mm_Vertical
- L1: footprint (none) -> Inductor_SMD:L_1008_2520Metric
- R1, R2, R3, R4, R5, R6: footprint (none) -> Resistor_SMD:R_0805_2012Metric
Connections:
- net GND: now also J1.2, J1.3
- net VIN: now also J1.1
Other:
- note added: "I presume that the tabel has a typo. C6's Unit is pF and not uF"
- note removed: "Thus, I presume that the tabel has a typo. C6's Unit is pF and not uF"

Commit message: redo component placement and finish routing
Parts:
- J2: footprint Connector_PinHeader_1.00mm:PinHeader_1x02_P1.00mm_Vertical -> Connector_PinHeader_2.00mm:PinHeader_1x02_P2.00mm_Vertical
Changed lines of the file:
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@@
 			)
 		)
-		(property "Footprint" "Connector_PinHeader_1.00mm:PinHeader_1x02_P1.00mm_Vertical"
+		(property "Footprint" "Connector_PinHeader_2.00mm:PinHeader_1x02_P2.00mm_Vertical"
 			(at 166.37 105.41 0)
 			(hide yes)
